File: 6gend-mb1.kicad_pcb (KiCad board)
At the start: 4 copper layers, 65 x 65 mm, 61 parts, among them J1 DEBUG, J2 SENSE, J3 POWER, J4 ACTUATE, J5 STORAGE, J6 JTAG, J7 RF, U1 STM32U031F8, Y1 32.768kHz

Commit message: Layout finished and ready for production.
Parts:
- moved R5 23.8 mm to (143.0, 102.0), turned to 180 degrees
- moved R4 15.6 mm to (143.1, 97.1), turned to 180 degrees
- moved TP5 10.2 mm to (143.0, 104.6)
- moved R6 4.68 mm to (155.6, 91.1), turned to -90 degrees
- moved TP4 2.54 mm to (143.0, 94.4)
- moved C3 2.06 mm to (143.8, 98.7)
- moved U1 2.06 mm to (152.8, 99.2)
- moved Y1 2.06 mm to (146.8, 99.4)
- moved C12 2.06 mm to (145.5, 103.1)
- moved C8 2.06 mm to (145.5, 96.1)
- moved C11 2.06 mm to (147.4, 103.1)
- moved C4 2.06 mm to (143.8, 100.3)
- moved C7 2.06 mm to (147.3, 96.1)
- moved R1 1.40 mm to (138.0, 83.4)
- moved R7 1.12 mm to (160.8, 83.4)
Routing:
- net VCC: track 0.00 -> 307.7 mm, vias 0 -> 25
- net VBAT: track 0.00 -> 189.6 mm, vias 0 -> 2
- net /SCL: track 0.00 -> 127.4 mm, vias 0 -> 10
- net /SDA: track 0.00 -> 124.8 mm, vias 0 -> 8
- net /SCK: track 0.00 -> 94.8 mm, vias 0 -> 2
- net /MOSI: track 0.00 -> 91.4 mm, vias 0 -> 2
- net /MISO: track 0.00 -> 90.4 mm, vias 0 -> 2
- net /LS1: track 0.00 -> 46.9 mm, vias 0 -> 4
- net /CS3: track 0.00 -> 42.8 mm, vias 0 -> 4
- net /PF3: track 0.00 -> 41.5 mm, vias 0 -> 2
- net /PWM: track 0.00 -> 32.5 mm, vias 0 -> 3
- net /CS1: track 0.00 -> 31.1 mm, vias 0 -> 4
- net /TxD: track 0.00 -> 29.8 mm
- net /RxD: track 0.00 -> 29.2 mm
- net /CS2: track 0.00 -> 28.9 mm
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- added copper zone on B.Cu, net GND
Other:
- copper layers 4 -> 2
- board text added: "A"
- board text added: "VCC range 1.7 - 3.6 V"
- board text removed: "a"
